Commit message: added STL files

File: cheetah_description/xacro/mini_cheetah.urdf (robot description, URDF)
Before this commit: robot mini_cheetah, 17 links, 16 joints
Links:
- link FL_calf: geometry collision mesh filename=package://cheetah_description/meshes/mini_lower_link.stl; visual mesh filename=package://cheetah_description/meshes/mini_lower_link.stl
- link FL_hip: geometry collision mesh filename=package://cheetah_description/meshes/mini_abad.stl; visual mesh filename=package://cheetah_description/meshes/mini_abad.stl
- link FL_thigh: geometry collision mesh filename=package://cheetah_description/meshes/mini_upper_link.stl; visual mesh filename=package://cheetah_description/meshes/mini_upper_link.stl
- link FR_calf: geometry collision mesh filename=package://cheetah_description/meshes/mini_lower_link.stl; visual mesh filename=package://cheetah_description/meshes/mini_lower_link.stl
- link FR_hip: geometry collision mesh filename=package://cheetah_description/meshes/mini_abad.stl; visual mesh filename=package://cheetah_description/meshes/mini_abad.stl
- link FR_thigh: geometry collision mesh filename=package://cheetah_description/meshes/mini_upper_link.stl; visual mesh filename=package://cheetah_description/meshes/mini_upper_link.stl
- link RL_calf: geometry collision mesh filename=package://cheetah_description/meshes/mini_lower_link.stl; visual mesh filename=package://cheetah_description/meshes/mini_lower_link.stl
- link RL_hip: geometry collision mesh filename=package://cheetah_description/meshes/mini_abad.stl; visual mesh filename=package://cheetah_description/meshes/mini_abad.stl
- link RL_thigh: geometry collision mesh filename=package://cheetah_description/meshes/mini_upper_link.stl; visual mesh filename=package://cheetah_description/meshes/mini_upper_link.stl
- link RR_calf: geometry collision mesh filename=package://cheetah_description/meshes/mini_lower_link.stl; visual mesh filename=package://cheetah_description/meshes/mini_lower_link.stl
- link RR_hip: geometry collision mesh filename=package://cheetah_description/meshes/mini_abad.stl; visual mesh filename=package://cheetah_description/meshes/mini_abad.stl
- link RR_thigh: geometry collision mesh filename=package://cheetah_description/meshes/mini_upper_link.stl; visual mesh filename=package://cheetah_description/meshes/mini_upper_link.stl
- link trunk: geometry collision mesh filename=package://cheetah_description/meshes/mini_body.stl; visual mesh filename=package://cheetah_description/meshes/mini_body.stl

Commit message: updated files

File: cheetah_description/xacro/mini_cheetah.urdf (robot description, URDF)
Before this commit: robot mini_cheetah, 17 links, 16 joints
Links:
- link FL_calf: mass 0.064 -> 0.1
- link FL_hip: mass 0.54 -> 0.05
- link FL_thigh: mass 0.634 -> 0.8
- link FR_calf: mass 0.064 -> 0.1
- link FR_hip: mass 0.54 -> 0.05
- link FR_thigh: mass 0.634 -> 0.8
- link RL_calf: mass 0.064 -> 0.1
- link RL_hip: mass 0.54 -> 0.05
- link RL_thigh: mass 0.634 -> 0.8
- link RR_calf: mass 0.064 -> 0.1
- link RR_hip: mass 0.54 -> 0.05
- link RR_thigh: mass 0.634 -> 0.8
- link trunk: mass 3.3 -> 2.1

Commit message: updated the urdf model

File: cheetah_description/xacro/mini_cheetah.urdf (robot description, URDF)
Before this commit: robot mini_cheetah, 17 links, 16 joints
Links:
- added link trunk_interia, mass 3.3; collision box size=0.3 0.2 0.093; visual mesh filename=package://cheetah_description/meshes/trunk.STL scale=1 1 1
- link FL_calf: mass 0.1 -> 0.064; geometry collision box size=0.016 0.016 0.2; visual mesh filename=package://cheetah_description/meshes/calf.STL scale=1 1 1
- link FL_foot: geometry collision sphere radius=0.025; visual mesh filename=package://cheetah_description/meshes/foot.STL scale=1 1 1
- link FL_hip: mass 0.05 -> 0.57; geometry collision box size=0.09 0.08 0.093; visual mesh filename=package://cheetah_description/meshes/hip.STL scale=1 1 1
- link FL_thigh: mass 0.8 -> 0.634; geometry collision box size=0.043 0.034 0.22; visual mesh filename=package://cheetah_description/meshes/thigh.STL scale=1 1 1
- link FR_calf: mass 0.1 -> 0.064; geometry collision box size=0.016 0.016 0.2; visual mesh filename=package://cheetah_description/meshes/calf.STL scale=1 1 1
- link FR_foot: geometry collision sphere radius=0.025; visual mesh filename=package://cheetah_description/meshes/foot.STL scale=1 1 1
- link FR_hip: mass 0.05 -> 0.57; geometry collision box size=0.09 0.08 0.093; visual mesh filename=package://cheetah_description/meshes/hip.STL scale=1 1 1
- link FR_thigh: mass 0.8 -> 0.634; geometry collision box size=0.043 0.034 0.22; visual mesh filename=package://cheetah_description/meshes/thigh.STL scale=1 1 1
- link RL_calf: mass 0.1 -> 0.064; geometry collision box size=0.016 0.016 0.2; visual mesh filename=package://cheetah_description/meshes/calf.STL scale=1 1 1
- link RL_foot: geometry collision sphere radius=0.025; visual mesh filename=package://cheetah_description/meshes/foot.STL scale=1 1 1
- link RL_hip: mass 0.05 -> 0.57; geometry collision box size=0.09 0.08 0.093; visual mesh filename=package://cheetah_description/meshes/hip.STL scale=1 1 1
- link RL_thigh: mass 0.8 -> 0.634; geometry collision box size=0.043 0.034 0.22; visual mesh filename=package://cheetah_description/meshes/thigh.STL scale=1 1 1
- link RR_calf: mass 0.1 -> 0.064; geometry collision box size=0.016 0.016 0.2; visual mesh filename=package://cheetah_description/meshes/calf.STL scale=1 1 1
- link RR_foot: geometry collision sphere radius=0.025; visual mesh filename=package://cheetah_description/meshes/foot.STL scale=1 1 1
- link RR_hip: mass 0.05 -> 0.57; geometry collision box size=0.09 0.08 0.093; visual mesh filename=package://cheetah_description/meshes/hip.STL scale=1 1 1
- link RR_thigh: mass 0.8 -> 0.634; geometry collision box size=0.043 0.034 0.22; visual mesh filename=package://cheetah_description/meshes/thigh.STL scale=1 1 1
- link trunk: mass 2.1 -> None; geometry 
Joints:
- added joint trunk_to_trunk_inertia: type fixed, parent trunk, child trunk_interia, origin xyz=0 0 0 rpy=0 0 0
- joint FL_calf_joint: limit (none) -> lower=-3.14159265359 upper=3.14159265359 effort=20 velocity=10.6; origin xyz=0 0 -0.209 rpy=0.0 0 0.0 -> xyz=0 0 -0.2115 rpy=0 0 0; type continuous -> revolute
- joint FL_foot_fixed: origin xyz=0 0 -0.18 -> xyz=0 0 -0.23039 rpy=0 0 0
- joint FL_hip_joint: limit (none) -> lower=-0.872664625997 upper=1.0471975512 effort=20 velocity=10.6; origin xyz=0.19 0.049 0.0 rpy=0 0 0 -> xyz=0.196 0.049664 0 rpy=0 0 0; type continuous -> revolute
- joint FL_thigh_joint: limit (none) -> lower=-0.523598775598 upper=3.92699081699 effort=20 velocity=10.6; origin xyz=0 0.062 0 rpy=0.0 0 0.0 -> xyz=0 0.077476 0 rpy=0 0 0; type continuous -> revolute
- joint FR_calf_joint: limit (none) -> lower=-3.14159265359 upper=3.14159265359 effort=20 velocity=10.6; origin xyz=0 0 -0.209  rpy=0.0 0 0.0 -> xyz=0 0 -0.2115 rpy=0 0 0; type continuous -> revolute
- joint FR_foot_fixed: origin xyz=0 0 -0.18 -> xyz=0 0 -0.23039 rpy=0 0 0
- joint FR_hip_joint: limit (none) -> lower=-1.0471975512 upper=0.872664625997 effort=20 velocity=10.6; origin xyz=0.19 -0.049 0.0 rpy=0 0 0 -> xyz=0.196 -0.049664 0 rpy=0 0 0; type continuous -> revolute
- joint FR_thigh_joint: limit (none) -> lower=-0.523598775598 upper=3.92699081699 effort=20 velocity=10.6; origin xyz=0 -0.062 0 rpy=0.0 0.0 0.0 -> xyz=0 -0.077476 0 rpy=0 0 0; type continuous -> revolute
- joint RL_calf_joint: limit (none) -> lower=-3.14159265359 upper=3.14159265359 effort=20 velocity=10.6; origin xyz=0 0 -0.209  rpy=0.0 0 0.0 -> xyz=0 0 -0.2115 rpy=0 0 0; type continuous -> revolute
- joint RL_foot_fixed: origin xyz=0 0 -0.18 -> xyz=0 0 -0.23039 rpy=0 0 0
- joint RL_hip_joint: limit (none) -> lower=-0.872664625997 upper=1.0471975512 effort=20 velocity=10.6; origin xyz=-0.19 0.049 0.0 rpy=0 0 0 -> xyz=-0.196 0.049664 0 rpy=0 0 0; type continuous -> revolute
- joint RL_thigh_joint: limit (none) -> lower=-0.523598775598 upper=3.92699081699 effort=20 velocity=10.6; origin xyz=0 0.062 0 rpy=0.0 0.0 0.0 -> xyz=0 0.077476 0 rpy=0 0 0; type continuous -> revolute
- joint RR_calf_joint: limit (none) -> lower=-3.14159265359 upper=3.14159265359 effort=20 velocity=10.6; origin xyz=0 0 -0.209  rpy=0.0 0 0.0 -> xyz=0 0 -0.2115 rpy=0 0 0; type continuous -> revolute
- joint RR_foot_fixed: origin xyz=0 0 -0.18 -> xyz=0 0 -0.23039 rpy=0 0 0
- joint RR_hip_joint: limit (none) -> lower=-1.0471975512 upper=0.872664625997 effort=20 velocity=10.6; origin xyz=-0.19 -0.049 0.0 rpy=0 0 0 -> xyz=-0.196 -0.049664 0 rpy=0 0 0; type continuous -> revolute
- joint RR_thigh_joint: limit (none) -> lower=-0.523598775598 upper=3.92699081699 effort=20 velocity=10.6; origin xyz=0 -0.062 0 rpy=0.0 0 0.0 -> xyz=0 -0.077476 0 rpy=0 0 0; type continuous -> revolute
